File: eagle/a3640.sch (EAGLE design)
At the start: 0 parts

Commit message: placed an 040 part and wired up the data/address buses to a net.
Parts:
- added IC1: MC68040RC, MC68K:MC68040RC
Connections:
- new net A040_0: IC1>NAME.A0
- new net A040_1: IC1>NAME.A1
- new net A040_10: IC1>NAME.A10
- new net A040_11: IC1>NAME.A11
- new net A040_12: IC1>NAME.A12
- new net A040_13: IC1>NAME.A13
- new net A040_14: IC1>NAME.A14
- new net A040_15: IC1>NAME.A15
- new net A040_16: IC1>NAME.A16
- new net A040_17: IC1>NAME.A17
- new net A040_18: IC1>NAME.A18
- new net A040_19: IC1>NAME.A19
- new net A040_2: IC1>NAME.A2
- new net A040_20: IC1>NAME.A20
- new net A040_21: IC1>NAME.A21
- new net A040_22: IC1>NAME.A22
- new net A040_23: IC1>NAME.A23
- new net A040_24: IC1>NAME.A24
- new net A040_25: IC1>NAME.A25
- new net A040_26: IC1>NAME.A26
- new net A040_27: IC1>NAME.A27
- new net A040_28: IC1>NAME.A28
- new net A040_29: IC1>NAME.A29
- new net A040_3: IC1>NAME.A3
- new net A040_30: IC1>NAME.A30
- new net A040_31: IC1>NAME.A31
- new net A040_4: IC1>NAME.A4
- new net A040_5: IC1>NAME.A5
- new net A040_6: IC1>NAME.A6
- new net A040_7: IC1>NAME.A7
- new net A040_8: IC1>NAME.A8
- new net A040_9: IC1>NAME.A9
- new net D040_0: IC1>NAME.D0
- new net D040_1: IC1>NAME.D1
- new net D040_10: IC1>NAME.D10
- new net D040_11: IC1>NAME.D11
- new net D040_12: IC1>NAME.D12
- new net D040_13: IC1>NAME.D13
- new net D040_14: IC1>NAME.D14
- new net D040_15: IC1>NAME.D15
- new net D040_16: IC1>NAME.D16
- new net D040_17: IC1>NAME.D17
- new net D040_18: IC1>NAME.D18
- new net D040_19: IC1>NAME.D19
- new net D040_2: IC1>NAME.D2
- new net D040_20: IC1>NAME.D20
- new net D040_21: IC1>NAME.D21
- new net D040_22: IC1>NAME.D22
- new net D040_23: IC1>NAME.D23
- new net D040_24: IC1>NAME.D24
- new net D040_25: IC1>NAME.D25
- new net D040_26: IC1>NAME.D26
- new net D040_27: IC1>NAME.D27
- new net D040_28: IC1>NAME.D28
- new net D040_29: IC1>NAME.D29
- new net D040_3: IC1>NAME.D3
- new net D040_30: IC1>NAME.D30
- new net D040_31: IC1>NAME.D31
- new net D040_4: IC1>NAME.D4
- new net D040_5: IC1>NAME.D5
- new net D040_6: IC1>NAME.D6
- new net D040_7: IC1>NAME.D7
- new net D040_8: IC1>NAME.D8
- new net D040_9: IC1>NAME.D9

Commit message: chipping away at the schematic
Connections:
- new net AVEC: IC1>NAME.!AVEC
- new net BB: IC1>NAME.!BB
- new net BCLK: IC1>NAME.BCLK
- new net BG: IC1>NAME.!BG
- new net BR: IC1>NAME.!BR
- new net IPL0: IC1>NAME.IPL0
- new net IPL1: IC1>NAME.IPL1
- new net IPL2: IC1>NAME.IPL2
- new net PCLK: IC1>NAME.PCLK
- new net R/W: IC1>NAME.R/!W
- new net SIZ0: IC1>NAME.SIZ0
- new net SIZ1: IC1>NAME.SIZ1
- new net TLN0: IC1>NAME.TLN0
- new net TLN1: IC1>NAME.TLN1
- new net TM0: IC1>NAME.TM0
- new net TM1: IC1>NAME.TM1
- new net TM2: IC1>NAME.TM2
- new net TT0: IC1>NAME.TT0
- new net TT1: IC1>NAME.TT1
Changed lines of the file:
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@@
 </instances>
 <busses>
-<bus name="VCC,GND,D040_[0..31],A040_[0..31]">
+<bus name="VCC,GND,D040_[0..31],A040_[0..31],IPL[0..2],BR,BG,BB,BCLK,PCLK,TT[0..1],TM[0..2],TLN[0..1],SIZ[0..1],R/W,AVEC">
 <segment>
 <wire x1="0" y1="0" x2="0" y2="215.9" width="0.762" layer="92"/>
@@
 </segment>
 </net>
+<net name="IPL0" class="0">
+<segment>
+<pinref part="IC1" gate="&gt;NAME" pin="IPL0"/>
+<wire x1="127" y1="132.08" x2="81.28" y2="132.08" width="0.1524" layer="91"/>
+<label x="99.06" y="132.08" size="1.778" layer="95"/>
+</segment>
+</net>
+<net name="IPL1" class="0">
+<segment>
+<pinref part="IC1" gate="&gt;NAME" pin="IPL1"/>
+<wire x1="127" y1="129.54" x2="81.28" y2="129.54" width="0.1524" layer="91"/>
+<label x="99.06" y="129.54" size="1.778" layer="95"/>
+</segment>
+</net>
+<net name="IPL2" class="0">
+<segment>
+<pinref part="IC1" gate="&gt;NAME" pin="IPL2"/>
+<wire x1="127" y1="127" x2="81.28" y2="127" width="0.1524" layer="91"/>
+<label x="99.06" y="127" size="1.778" layer="95"/>
+</segment>
+</net>
+<net name="BR" class="0">
+<segment>
+<pinref part="IC1" gate="&gt;NAME" pin="!BR"/>
+<wire x1="127" y1="154.94" x2="81.28" y2="154.94" width="0.1524" layer="91"/>
+<label x="99.06" y="154.94" size="1.778" layer="95"/>
+</segment>
+</net>
+<net name="BG" class="0">
+<segment>
+<pinref part="IC1" gate="&gt;NAME" pin="!BG"/>
+<wire x1="127" y1="152.4" x2="81.28" y2="152.4" width="0.1524" layer="91"/>
+<label x="99.06" y="152.4" size="1.778" layer="95"/>
+</segment>
+</net>
+<net name="BB" class="0">
+<segment>
+<pinref part="IC1" gate="&gt;NAME" pin="!BB"/>
+<wire x1="127" y1="149.86" x2="81.28" y2="149.86" width="0.1524" layer="91"/>
+<label x="99.06" y="149.86" size="1.778" layer="95"/>
+</segment>
+</net>
+<net name="BCLK" class="0">
+<segment>
+<pinref part="IC1" gate="&gt;NAME" pin="BCLK"/>
+<wire x1="0" y1="177.8" x2="45.72" y2="177.8" width="0.1524" layer="91"/>
+<label x="17.78" y="177.8" size="1.778" layer="95"/>
+</segment>
+</net>
+<net name="PCLK" class="0">
+<segment>
+<pinref part="IC1" gate="&gt;NAME" pin="PCLK"/>
+<wire x1="0" y1="172.72" x2="45.72" y2="172.72" width="0.1524" layer="91"/>
+<label x="17.78" y="172.72" size="1.778" layer="95"/>
+</segment>
+</net>
+<net name="TT0" class="0">
+<segment>
+<pinref part="IC1" gate="&gt;NAME" pin="TT0"/>
+<wire x1="0" y1="167.64" x2="45.72" y2="167.64" width="0.1524" layer="91"/>
+<label x="17.78" y="167.64" size="1.778" layer="95"/>
+</segment>
+</net>
+<net name="TT1" class="0">
+<segment>
+<pinref part="IC1" gate="&gt;NAME" pin="TT1"/>
+<wire x1="0" y1="165.1" x2="45.72" y2="165.1" width="0.1524" layer="91"/>
+<label x="17.78" y="165.1" size="1.778" layer="95"/>
+</segment>
+</net>
+<net name="TM0" class="0">
+<segment>
+<pinref part="IC1" gate="&gt;NAME" pin="TM0"/>
+<wire x1="0" y1="162.56" x2="45.72" y2="162.56" width="0.1524" layer="91"/>
+<label x="17.78" y="162.56" size="1.778" layer="95"/>
+</segment>
+</net>
+<net name="TM1" class="0">
+<segment>
+<pinref part="IC1" gate="&gt;NAME" pin="TM1"/>
+<wire x1="0" y1="160.02" x2="45.72" y2="160.02" width="0.1524" layer="91"/>
+<label x="17.78" y="160.02" size="1.778" layer="95"/>
+</segment>
+</net>
+<net name="TM2" class="0">
+<segment>
+<pinref part="IC1" gate="&gt;NAME" pin="TM2"/>
+<wire x1="0" y1="157.48" x2="45.72" y2="157.48" width="0.1524" layer="91"/>
+<label x="17.78" y="157.48" size="1.778" layer="95"/>
+</segment>
+</net>
+<net name="TLN0" class="0">
+<segment>
+<pinref part="IC1" gate="&gt;NAME" pin="TLN0"/>
+<wire x1="0" y1="154.94" x2="45.72" y2="154.94" width="0.1524" layer="91"/>
+<label x="17.78" y="154.94" size="1.778" layer="95"/>
+</segment>
+</net>
+<net name="TLN1" class="0">
+<segment>
+<pinref part="IC1" gate="&gt;NAME" pin="TLN1"/>
+<wire x1="0" y1="152.4" x2="45.72" y2="152.4" width="0.1524" layer="91"/>
+<label x="17.78" y="152.4" size="1.778" layer="95"/>
+</segment>
+</net>
+<net name="SIZ0" class="0">
+<segment>
+<pinref part="IC1" gate="&gt;NAME" pin="SIZ0"/>
+<wire x1="0" y1="142.24" x2="45.72" y2="142.24" width="0.1524" layer="91"/>
+<label x="17.78" y="142.24" size="1.778" layer="95"/>
+</segment>
+</net>
+<net name="SIZ1" class="0">
+<segment>
+<pinref part="IC1" gate="&gt;NAME" pin="SIZ1"/>
+<wire x1="0" y1="139.7" x2="45.72" y2="139.7" width="0.1524" layer="91"/>
+<label x="17.78" y="139.7" size="1.778" layer="95"/>
+</segment>
+</net>
+<net name="R/W" class="0">
+<segment>
+<pinref part="IC1" gate="&gt;NAME" pin="R/!W"/>
+<wire x1="0" y1="144.78" x2="45.72" y2="144.78" width="0.1524" layer="91"/>
+<label x="17.78" y="144.78" size="1.778" layer="95"/>
+</segment>
+</net>
+<net name="AVEC" class="0">
+<segment>
+<pinref part="IC1" gate="&gt;NAME" pin="!AVEC"/>
+<wire x1="127" y1="119.38" x2="81.28" y2="119.38" width="0.1524" layer="91"/>
+<label x="99.06" y="119.38" size="1.778" layer="95"/>
+</segment>
+</net>

Commit message: More stuff.
Parts:
- added U214, U215, U216, U217, U218, U219, U220, U221: 74FCT543, terriblefire:74FCT543
Connections:
- net D040_0: now also U218.A0, U219.A0, U220.A0
- net D040_1: now also U218.A1, U219.A1, U220.A1
- net D040_10: now also U217.A2, U221.A2
- net D040_11: now also U217.A3, U221.A3
- net D040_12: now also U217.A4, U221.A4
- net D040_13: now also U217.A5, U221.A5
- net D040_14: now also U217.A6, U221.A6
- net D040_15: now also U217.A7, U221.A7
- net D040_16: now also U215.A0, U216.A0
- net D040_17: now also U215.A1, U216.A1
- net D040_18: now also U215.A2, U216.A2
- net D040_19: now also U215.A3, U216.A3
- net D040_2: now also U218.A2, U219.A2, U220.A2
- net D040_20: now also U215.A4, U216.A4
- net D040_21: now also U215.A5, U216.A5
- net D040_22: now also U215.A6, U216.A6
- net D040_23: now also U215.A7, U216.A7
- net D040_24: now also U214.A0
- net D040_25: now also U214.A1
- net D040_26: now also U214.A2
- net D040_27: now also U214.A3
- net D040_28: now also U214.A4
- net D040_29: now also U214.A5
- net D040_3: now also U218.A3, U219.A3, U220.A3
- net D040_30: now also U214.A6
- net D040_31: now also U214.A7
- net D040_4: now also U218.A4, U219.A4, U220.A4
- net D040_5: now also U218.A5, U219.A5, U220.A5
- net D040_6: now also U218.A6, U219.A6, U220.A6
- net D040_7: now also U218.A7, U219.A7, U220.A7
- net D040_8: now also U217.A0, U221.A0
- net D040_9: now also U217.A1, U221.A1

Commit message: footprint update and parts placement
Parts:
- added U204, U205, U207, U209: GAL22V10, a3640_edu_v0.1:GAL22V10
- U214, U215, U216, U217, U218, U219, U220, U221: value 74FCT543 -> 74FCT543SOIC24; device terriblefire:74FCT543 -> terriblefire:74FCT543SOIC24
Changed lines of the file:
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@@
 <parts>
 <part name="IC1" library="MC68K" deviceset="MC68040RC" device=""/>
-<part name="U214" library="terriblefire" deviceset="74FCT543" device=""/>
-<part name="U215" library="terriblefire" deviceset="74FCT543" device=""/>
-<part name="U216" library="terriblefire" deviceset="74FCT543" device=""/>
-<part name="U217" library="terriblefire" deviceset="74FCT543" device=""/>
-<part name="U218" library="terriblefire" deviceset="74FCT543" device=""/>
-<part name="U219" library="terriblefire" deviceset="74FCT543" device=""/>
-<part name="U220" library="terriblefire" deviceset="74FCT543" device=""/>
-<part name="U221" library="terriblefire" deviceset="74FCT543" device=""/>
+<part name="U214" library="terriblefire" deviceset="74FCT543" device="SOIC24" value="74FCT543SOIC24"/>
+<part name="U215" library="terriblefire" deviceset="74FCT543" device="SOIC24" value="74FCT543SOIC24"/>
+<part name="U216" library="terriblefire" deviceset="74FCT543" device="SOIC24" value="74FCT543SOIC24"/>
+<part name="U217" library="terriblefire" deviceset="74FCT543" device="SOIC24" value="74FCT543SOIC24"/>
+<part name="U218" library="terriblefire" deviceset="74FCT543" device="SOIC24" value="74FCT543SOIC24"/>
+<part name="U219" library="terriblefire" deviceset="74FCT543" device="SOIC24" value="74FCT543SOIC24"/>
+<part name="U220" library="terriblefire" deviceset="74FCT543" device="SOIC24" value="74FCT543SOIC24"/>
+<part name="U221" library="terriblefire" deviceset="74FCT543" device="SOIC24" value="74FCT543SOIC24"/>
+<part name="U204" library="a3640_edu_v0.1" deviceset="GAL22V10" device=""/>
+<part name="U205" library="a3640_edu_v0.1" deviceset="GAL22V10" device=""/>
+<part name="U209" library="a3640_edu_v0.1" deviceset="GAL22V10" device=""/>
+<part name="U207" library="a3640_edu_v0.1" deviceset="GAL22V10" device=""/>
 </parts>
 <sheets>
@@
 </instances>
 <busses>
-<bus name="VCC,GND,D040_[0..31],A040_[0..31],IPL[0..2],BR,BG,BB,BCLK,PCLK,TT[0..1],TM[0..2],TLN[0..1],SIZ[0..1],R/W,AVEC,LEBUS[0..7]">
+<bus name="VCC,GND,D[0..31],D040_[0..31],A040_[0..31],IPL[0..2],BR,BG,BB,BCLK,PCLK,TT[0..1],TM[0..2],TLN[0..1],SIZ[0..1],R/W,AVEC,LEBUS[0..7]">
 <segment>
 <wire x1="0" y1="0" x2="0" y2="132.08" width="0.762" layer="92"/>
@@
 </nets>
 </sheet>
+<sheet>
+<plain>
+</plain>
+<instances>
+<instance part="U204" gate="G$1" x="71.12" y="137.16"/>
+<instance part="U205" gate="G$1" x="71.12" y="66.04"/>
+<instance part="U209" gate="G$1" x="167.64" y="134.62"/>
+<instance part="U207" gate="G$1" x="167.64" y="66.04"/>
+</instances>
+<busses>
+</busses>
+<nets>
+</nets>
+</sheet>
